File: Hardware/VoltageReferenceProgrammableRevD.brd (EAGLE design)
At the start: 69.8 x 31.8 mm, 57 parts, among them J1 AVR_SPI_PRG_6PTH, J2 POWER_JACKPTH, U1 MIC5205, U2 REF5040ID, U3 ATMEGA328, U4 SN74LV164APW, U5 AD5040BRJZ, U6 OPA365, Y1 16MHz

Commit message: Corrected error on schematic & BOM
AD5040 was replaced with AD5060.
Parts:
- U5: value AD5040BRJZ -> AD5060BRJZ
